Commit message: Update skid-steer robot model and SBG configuration

File: src/my_robot_description/urdf/robot.urdf.xacro (robot description, xacro)
@@ -1,20 +1,40 @@
 <?xml version="1.0"?>
 <robot xmlns:xacro="http://www.ros.org/wiki/xacro"
-       name="four_wheel_robot">
-  <!-- 颜色 -->
+       name="agricultural_skid_steer_robot">
+  <!-- ====================================================== -->
+  <!-- Robot geometry parameters                              -->
+  <!-- ====================================================== -->
+  <!-- Current measured geometry -->
+  <!-- Track width may be updated after chassis modification -->
+  <xacro:property name="wheelbase" value="1.07"/>
+  <xacro:property name="track_width" value="0.55"/>
+  <xacro:property name="wheel_radius" value="0.22"/>
+  <xacro:property name="wheel_width" value="0.11"/>
+  <!--
+    Temporary chassis visualization dimensions.
+    These are NOT the skid-steer kinematic dimensions.
+    Update after final mechanical modification.
+  -->
+  <xacro:property name="base_length" value="1.20"/>
+  <xacro:property name="base_width" value="0.50"/>
+  <xacro:property name="base_height" value="0.20"/>
+  <!-- ====================================================== -->
+  <!-- Materials                                              -->
+  <!-- ====================================================== -->
   <material name="blue">
-    <color rgba="0.1 0.4 0.8 1.0"/>
+    <color rgba="0.1 0.3 0.8 1.0"/>
   </material>
   <material name="black">
     <color rgba="0.05 0.05 0.05 1.0"/>
   </material>
-  <!-- 地面参考坐标系 -->
+  <!-- ====================================================== -->
+  <!-- Base frames                                            -->
+  <!-- ====================================================== -->
   <link name="base_footprint"/>
-  <!-- 机器人底盘 -->
   <link name="base_link">
     <visual>
       <origin xyz="0 0 0" rpy="0 0 0"/>
       <geometry>
-        <box size="1.0 0.65 0.20"/>
+        <box size="${base_length} ${base_width} ${base_height}"/>
       </geometry>
       <material name="blue"/>
@@ -23,5 +43,5 @@
       <origin xyz="0 0 0" rpy="0 0 0"/>
       <geometry>
-        <box size="1.0 0.65 0.20"/>
+        <box size="${base_length} ${base_width} ${base_height}"/>
       </geometry>
     </collision>
@@ -29,47 +49,52 @@
       <origin xyz="0 0 0" rpy="0 0 0"/>
       <mass value="20.0"/>
+      <!-- Temporary inertia values -->
       <inertia
-        ixx="0.7708"
+        ixx="1.0"
         ixy="0.0"
         ixz="0.0"
-        iyy="1.7333"
+        iyy="2.5"
         iyz="0.0"
-        izz="2.4375"/>
+        izz="3.0"/>
     </inertial>
   </link>
-  <!-- 把底盘安装在地面参考坐标系上方 -->
+  <!--
+    base_link origin is approximately at the chassis geometric center.
+    With a 0.22 m wheel radius and 0.20 m chassis height,
+    this temporary height places the wheels near the ground plane.
+  -->
   <joint name="base_footprint_joint" type="fixed">
     <parent link="base_footprint"/>
     <child link="base_link"/>
-    <origin xyz="0 0 0.25" rpy="0 0 0"/>
-  </joint>
-  <!-- 四轮独立转向组件 -->
-  <xacro:macro name="wheel_assembly" params="prefix x y">
-    <!-- 转向架 -->
-    <link name="${prefix}_steering_link"/>
-    <!-- 转向关节：绕Z轴旋转 -->
-    <joint name="${prefix}_steering_joint" type="revolute">
-      <parent link="base_link"/>
-      <child link="${prefix}_steering_link"/>
-      <origin xyz="${x} ${y} -0.10" rpy="0 0 0"/>
-      <axis xyz="0 0 1"/>
-      <limit lower="-1.5708"
-             upper="1.5708"
-             effort="30.0"
-             velocity="1.5"/>
-    </joint>
-    <!-- 车轮 -->
+    <origin xyz="0 0 0.22" rpy="0 0 0"/>
+  </joint>
+  <!-- ====================================================== -->
+  <!-- Wheel macro                                            -->
+  <!-- ====================================================== -->
+  <!--
+    Four-wheel skid-steer configuration.
+    IMPORTANT:
+    The wheels do NOT steer around the Z axis.
+    Steering is generated by differential velocity between
+    the left and right wheel groups.
+  -->
+  <xacro:macro name="wheel" params="prefix x y">
     <link name="${prefix}_wheel_link">
       <visual>
-        <origin xyz="0 0 0" rpy="1.5708 0 0"/>
+        <!-- Cylinder axis converted to wheel axle direction -->
+        <origin xyz="0 0 0" rpy="1.57079632679 0 0"/>
         <geometry>
-          <cylinder radius="0.15" length="0.08"/>
+          <cylinder
+            radius="${wheel_radius}"
+            length="${wheel_width}"/>
         </geometry>
         <material name="black"/>
       </visual>
       <collision>
-        <origin xyz="0 0 0" rpy="1.5708 0 0"/>
+        <origin xyz="0 0 0" rpy="1.57079632679 0 0"/>
         <geometry>
-          <cylinder radius="0.15" length="0.08"/>
+          <cylinder
+            radius="${wheel_radius}"
+            length="${wheel_width}"/>
         </geometry>
       </collision>
@@ -77,27 +102,57 @@
         <origin xyz="0 0 0" rpy="0 0 0"/>
         <mass value="2.0"/>
+        <!-- Approximate wheel inertia -->
         <inertia
-          ixx="0.0123"
+          ixx="0.03"
           ixy="0.0"
           ixz="0.0"
-          iyy="0.0225"
+          iyy="0.05"
           iyz="0.0"
-          izz="0.0123"/>
+          izz="0.03"/>
       </inertial>
     </link>
-    <!-- 车轮绕Y轴滚动 -->
+    <!--
+      Wheel has ONLY rolling rotation.
+      No steering joint is present.
+    -->
     <joint name="${prefix}_wheel_joint" type="continuous">
-      <parent link="${prefix}_steering_link"/>
+      <parent link="base_link"/>
       <child link="${prefix}_wheel_link"/>
-      <origin xyz="0 0 0" rpy="0 0 0"/>
+      <origin
+        xyz="${x} ${y} 0"
+        rpy="0 0 0"/>
       <axis xyz="0 1 0"/>
     </joint>
   </xacro:macro>
-  <!-- 前左、前右、后左、后右 -->
-  <xacro:wheel_assembly prefix="front_left"  x="0.38"  y="0.365"/>
-  <xacro:wheel_assembly prefix="front_right" x="0.38"  y="-0.365"/>
-  <xacro:wheel_assembly prefix="rear_left"   x="-0.38" y="0.365"/>
-  <xacro:wheel_assembly prefix="rear_right"  x="-0.38" y="-0.365"/>
-    <!-- Gemini 335 深度相机 -->
+  <!-- ====================================================== -->
+  <!-- Four wheels                                            -->
+  <!-- ====================================================== -->
+  <!--
+    wheelbase   = 1.07 m  -> +/- 0.535 m
+    track_width = 0.55 m  -> +/- 0.275 m
+  -->
+  <xacro:wheel
+    prefix="front_left"
+    x="${wheelbase / 2.0}"
+    y="${track_width / 2.0}"/>
+  <xacro:wheel
+    prefix="front_right"
+    x="${wheelbase / 2.0}"
+    y="${-track_width / 2.0}"/>
+  <xacro:wheel
+    prefix="rear_left"
+    x="${-wheelbase / 2.0}"
+    y="${track_width / 2.0}"/>
+  <xacro:wheel
+    prefix="rear_right"
+    x="${-wheelbase / 2.0}"
+    y="${-track_width / 2.0}"/>
+  <!-- ====================================================== -->
+  <!-- Camera frame                                           -->
+  <!-- ====================================================== -->
+  <!--
+    Existing temporary camera transform.
+    Update later using actual measured sensor mounting position.
+  -->
   <link name="camera_link">
     <visual>
@@ -108,16 +163,42 @@
       <material name="black"/>
     </visual>
-    <collision>
-      <origin xyz="0 0 0" rpy="0 0 0"/>
-      <geometry>
-        <box size="0.04 0.115 0.025"/>
-      </geometry>
-    </collision>
   </link>
-  <!-- 相机安装在底盘前上方 -->
   <joint name="camera_joint" type="fixed">
     <parent link="base_link"/>
     <child link="camera_link"/>
-    <origin xyz="0.30 0 0.13" rpy="0 0 0"/>
-  </joint>
-  </robot>
+    <origin
+      xyz="0.30 0 0.13"
+      rpy="0 0 0"/>
+  </joint>
+  <!-- ====================================================== -->
+  <!-- SBG IMU frame                                          -->
+  <!-- ====================================================== -->
+  <!--
+    TEMPORARY extrinsic transform.
+    Measure actual SBG position/orientation before localization
+    experiments.
+  -->
+  <link name="imu_link"/>
+  <joint name="imu_joint" type="fixed">
+    <parent link="base_link"/>
+    <child link="imu_link"/>
+    <origin
+      xyz="0 0 0"
+      rpy="0 0 0"/>
+  </joint>
+  <!-- ====================================================== -->
+  <!-- GNSS main antenna frame                                -->
+  <!-- ====================================================== -->
+  <!--
+    TEMPORARY extrinsic transform.
+    Replace with measured main antenna phase-center position.
+  -->
+  <link name="gps_link"/>
+  <joint name="gps_joint" type="fixed">
+    <parent link="base_link"/>
+    <child link="gps_link"/>
+    <origin
+      xyz="0 0 0"
+      rpy="0 0 0"/>
+  </joint>
+</robot>

Commit message: AMIGA unified bringup and SLAM baseline

File: src/my_robot_description/urdf/robot.urdf.xacro (robot description, xacro)
@@ -16,6 +16,6 @@
     Update after final mechanical modification.
   -->
-  <xacro:property name="base_length" value="1.20"/>
-  <xacro:property name="base_width" value="0.50"/>
+  <xacro:property name="base_length" value="1.41"/>
+  <xacro:property name="base_width" value="0.80"/>
   <xacro:property name="base_height" value="0.20"/>
   <!-- ====================================================== -->
@@ -60,12 +60,17 @@
   </link>
   <!--
-    base_link origin is approximately at the chassis geometric center.
-    With a 0.22 m wheel radius and 0.20 m chassis height,
-    this temporary height places the wheels near the ground plane.
+    Coordinate convention:
+      X = forward
+      Y = left
+      Z = up
+    base_link origin is defined at the geometric center
+    of the SBG IMU.
+    Measured SBG center height above ground:
+      0.715 m
   -->
   <joint name="base_footprint_joint" type="fixed">
     <parent link="base_footprint"/>
     <child link="base_link"/>
-    <origin xyz="0 0 0.22" rpy="0 0 0"/>
+    <origin xyz="0 0 0.715" rpy="0 0 0"/>
   </joint>
   <!-- ====================================================== -->
@@ -149,11 +154,12 @@
     y="${-track_width / 2.0}"/>
   <!-- ====================================================== -->
-  <!-- Camera frame                                           -->
-  <!-- ====================================================== -->
-  <!--
-    Existing temporary camera transform.
-    Update later using actual measured sensor mounting position.
-  -->
-  <link name="camera_link">
+  <!-- Front camera frame                                           -->
+  <!-- ====================================================== -->
+  <!--
+    Temporary front camera transform.
+    Camera position may be changed after final mechanical
+    modification, so this transform is NOT final.
+  -->
+  <link name="front_camera_link">
     <visual>
       <origin xyz="0 0 0" rpy="0 0 0"/>
@@ -164,10 +170,34 @@
     </visual>
   </link>
-  <joint name="camera_joint" type="fixed">
-    <parent link="base_link"/>
-    <child link="camera_link"/>
-    <origin
-      xyz="0.30 0 0.13"
-      rpy="0 0 0"/>
+  <joint name="front_camera_joint" type="fixed">
+    <parent link="base_link"/>
+    <child link="front_camera_link"/>
+    <origin
+      xyz="0.56 0 0.58"
+      rpy="0 0.2618 0"/>
+  </joint>
+  <!-- ====================================================== -->
+  <!-- Rear camera frame                                      -->
+  <!-- ====================================================== -->
+  <!--
+    Temporary rear camera transform.
+    Position and approximately 15 degree downward tilt
+    are based on current mechanical installation.
+  -->
+  <link name="rear_camera_link">
+    <visual>
+      <origin xyz="0 0 0" rpy="0 0 0"/>
+      <geometry>
+        <box size="0.04 0.115 0.025"/>
+      </geometry>
+      <material name="black"/>
+    </visual>
+  </link>
+  <joint name="rear_camera_joint" type="fixed">
+    <parent link="base_link"/>
+    <child link="rear_camera_link"/>
+    <origin
+      xyz="-0.79 0 0.58"
+      rpy="0 -0.2618 3.14159"/>
   </joint>
   <!-- ====================================================== -->
@@ -175,15 +205,6 @@
   <!-- ====================================================== -->
   <!--
-    SBG IMU reference point.
-    SBG is located approximately at the chassis planar
-    geometric center.
-    Measured IMU reference height:
-      approximately 0.685 m above ground.
-    base_link height:
-      approximately 0.220 m above ground.
-    Therefore:
-      base_link -> imu_link z
-      = 0.685 - 0.220
-      = 0.465 m
+    base_link is defined at the SBG IMU geometric center.
+    Therefore imu_link is coincident with base_link.
   -->
   <link name="imu_link"/>
@@ -192,26 +213,17 @@
     <child link="imu_link"/>
     <origin
-      xyz="0 0 0.465"
-      rpy="0 0 0"/>
-  </joint>
-  <!-- ====================================================== -->
-  <!-- GNSS Primary antenna frame                             -->
-  <!-- ====================================================== -->
-  <!--
-    gps_link represents the ANT1 / Primary GNSS antenna
-    phase center.
-    Measured antenna geometry relative to the SBG IMU:
+      xyz="0 0 0"
+      rpy="0 0 0"/>
+  </joint>
+  <!-- ====================================================== -->
+  <!-- SBG GNSS primary antenna ANT1                          -->
+  <!-- ====================================================== -->
+  <!--
+    ANT1 / Primary GNSS antenna relative to the SBG center:
       X = +0.640 m forward
       Y =  0.000 m
-      Z = +0.685 m upward in ROS FLU coordinates
-    Therefore relative to base_link:
-      X = +0.640 m
-      Y =  0.000 m
-      Z = 0.465 + 0.685
-        = 1.150 m
-    The corresponding SBG internal lever arm is expressed
-    in the SBG body frame (X forward, Y right, Z down), so
-    its Z sign is negative there. Do not confuse the SBG
-    lever arm convention with ROS FLU coordinates.
+      Z = +0.685 m upward
+    ROS frame convention:
+      X forward, Y left, Z up
   -->
   <link name="gps_link"/>
@@ -220,5 +232,40 @@
     <child link="gps_link"/>
     <origin
-      xyz="0.640 0 1.150"
+      xyz="0.640 0 0.685"
+      rpy="0 0 0"/>
+  </joint>
+  <!-- ====================================================== -->
+  <!-- Independent white GNSS antenna                         -->
+  <!-- ====================================================== -->
+  <!--
+    Farm-ng white GNSS antenna relative to SBG/base_link:
+      X = +0.480 m
+      Y =  0.000 m
+      Z = +0.645 m
+  -->
+  <link name="white_gnss_link"/>
+  <joint name="white_gnss_joint" type="fixed">
+    <parent link="base_link"/>
+    <child link="white_gnss_link"/>
+    <origin
+      xyz="0.480 0 0.645"
+      rpy="0 0 0"/>
+  </joint>
+  <!-- ====================================================== -->
+  <!-- Velodyne VLP-16                                        -->
+  <!-- ====================================================== -->
+  <!--
+    Velodyne center relative to SBG/base_link:
+      X = +0.680 m
+      Y = +0.150 m
+      Z = +0.210 m
+    Positive Y is robot left side.
+  -->
+  <link name="velodyne"/>
+  <joint name="velodyne_joint" type="fixed">
+    <parent link="base_link"/>
+    <child link="velodyne"/>
+    <origin
+      xyz="0.680 0.150 0.210"
       rpy="0 0 0"/>
   </joint>

Commit message: Calibrate AMIGA localization and document SLAM bias

File: src/my_robot_description/urdf/robot.urdf.xacro (robot description, xacro)
@@ -70,7 +70,7 @@
   -->
   <joint name="base_footprint_joint" type="fixed">
-    <parent link="base_footprint"/>
-    <child link="base_link"/>
-    <origin xyz="0 0 0.715" rpy="0 0 0"/>
+    <parent link="base_link"/>
+    <child link="base_footprint"/>
+    <origin xyz="0 0 -0.715" rpy="0 0 0"/>
   </joint>
   <!-- ====================================================== -->
@@ -121,5 +121,5 @@
       No steering joint is present.
     -->
-    <joint name="${prefix}_wheel_joint" type="continuous">
+    <joint name="${prefix}_wheel_joint" type="fixed">
       <parent link="base_link"/>
       <child link="${prefix}_wheel_link"/>
@@ -127,5 +127,4 @@
         xyz="${x} ${y} 0"
         rpy="0 0 0"/>
-      <axis xyz="0 1 0"/>
     </joint>
   </xacro:macro>
@@ -268,5 +267,5 @@
     <origin
       xyz="0.680 0.150 0.210"
-      rpy="0 0 0"/>
+      rpy="0 0 -1.228"/>
   </joint>
 </robot>
